Commit message: Integrate DASE7503 Raspberry Pi ESP32 mecanum stack

File: src/mecanum_description/urdf/mecanum_amr.urdf.xacro (robot description, xacro)
@@ -2,14 +2,15 @@
 <robot name="mecanum_amr" xmlns:xacro="http://www.ros.org/wiki/xacro">
   <!-- ==================== Properties ==================== -->
-  <xacro:property name="base_width"  value="0.60"/>
-  <xacro:property name="base_length" value="0.80"/>
-  <xacro:property name="base_height" value="0.20"/>
-  <xacro:property name="base_mass"   value="50.0"/>
-  <xacro:property name="wheel_radius" value="0.075"/>
-  <xacro:property name="wheel_width"  value="0.05"/>
-  <xacro:property name="wheel_mass"   value="2.0"/>
-  <xacro:property name="wheel_x_offset" value="0.25"/>
-  <xacro:property name="wheel_y_offset" value="0.35"/>
-  <xacro:property name="wheel_z_offset" value="-0.05"/>
+  <!-- Safe starter dimensions only: replace with the measured acrylic chassis. -->
+  <xacro:property name="base_width"  value="0.27"/>
+  <xacro:property name="base_length" value="0.32"/>
+  <xacro:property name="base_height" value="0.06"/>
+  <xacro:property name="base_mass"   value="3.0"/>
+  <xacro:property name="wheel_radius" value="0.05"/>
+  <xacro:property name="wheel_width"  value="0.04"/>
+  <xacro:property name="wheel_mass"   value="0.15"/>
+  <xacro:property name="wheel_x_offset" value="0.115"/>
+  <xacro:property name="wheel_y_offset" value="0.125"/>
+  <xacro:property name="wheel_z_offset" value="-0.01"/>
   <!-- ==================== Macros ==================== -->
   <xacro:macro name="box_inertia" params="m w h d">
@@ -102,5 +103,5 @@
     <parent link="base_link"/>
     <child  link="lidar_link"/>
-    <origin xyz="0.3 0 ${base_height/2 + 0.035}" rpy="0 0 0"/>
+    <origin xyz="0 0 ${base_height/2 + 0.055}" rpy="0 0 0"/>
   </joint>
   <!-- LiDAR Gazebo plugin -->
@@ -155,5 +156,5 @@
     <parent link="base_link"/>
     <child  link="camera_link"/>
-    <origin xyz="0.35 0 ${base_height/2}" rpy="0 0 0"/>
+    <origin xyz="0.13 0 ${base_height/2 + 0.08}" rpy="0 0 0"/>
   </joint>
   <link name="camera_optical_link"/>
@@ -189,5 +190,5 @@
     <visual>
       <geometry>
-        <box size="0.50 0.40 0.02"/>
+        <box size="0.22 0.18 0.01"/>
       </geometry>
       <material name="orange">
@@ -197,8 +198,8 @@
     <collision>
       <geometry>
-        <box size="0.50 0.40 0.02"/>
-      </geometry>
-    </collision>
-    <xacro:box_inertia m="5.0" w="0.40" h="0.02" d="0.50"/>
+        <box size="0.22 0.18 0.01"/>
+      </geometry>
+    </collision>
+    <xacro:box_inertia m="0.25" w="0.18" h="0.01" d="0.22"/>
   </link>
   <joint name="lift_joint" type="prismatic">
@@ -207,5 +208,5 @@
     <origin xyz="0 0 ${base_height/2}" rpy="0 0 0"/>
     <axis xyz="0 0 1"/>
-    <limit lower="0.0" upper="0.30" effort="500" velocity="0.1"/>
+    <limit lower="0.0" upper="0.08" effort="50" velocity="0.05"/>
     <dynamics damping="10.0" friction="5.0"/>
   </joint>

Commit message: Refactor for course ESP32-S3 hardware

File: src/mecanum_description/urdf/mecanum_amr.urdf.xacro (robot description, xacro)
@@ -2,15 +2,17 @@
 <robot name="mecanum_amr" xmlns:xacro="http://www.ros.org/wiki/xacro">
   <!-- ==================== Properties ==================== -->
-  <!-- Safe starter dimensions only: replace with the measured acrylic chassis. -->
-  <xacro:property name="base_width"  value="0.27"/>
-  <xacro:property name="base_length" value="0.32"/>
-  <xacro:property name="base_height" value="0.06"/>
+  <!-- Clean-room model from the same-hardware profile; verify acrylic dimensions. -->
+  <xacro:property name="base_width"  value="0.18"/>
+  <xacro:property name="base_length" value="0.22"/>
+  <xacro:property name="base_height" value="0.04"/>
   <xacro:property name="base_mass"   value="3.0"/>
-  <xacro:property name="wheel_radius" value="0.05"/>
+  <!-- 150.8 mm measured circumference gives a 24.0 mm nominal radius. -->
+  <xacro:property name="wheel_radius" value="0.0240006"/>
   <xacro:property name="wheel_width"  value="0.04"/>
   <xacro:property name="wheel_mass"   value="0.15"/>
-  <xacro:property name="wheel_x_offset" value="0.115"/>
-  <xacro:property name="wheel_y_offset" value="0.125"/>
-  <xacro:property name="wheel_z_offset" value="-0.01"/>
+  <xacro:property name="wheel_x_offset" value="0.0475"/>
+  <xacro:property name="wheel_y_offset" value="0.0675"/>
+  <xacro:property name="wheel_z_offset" value="0.0"/>
+  <xacro:property name="lidar_z_offset" value="0.156"/>
   <!-- ==================== Macros ==================== -->
   <xacro:macro name="box_inertia" params="m w h d">
@@ -103,5 +105,5 @@
     <parent link="base_link"/>
     <child  link="lidar_link"/>
-    <origin xyz="0 0 ${base_height/2 + 0.055}" rpy="0 0 0"/>
+    <origin xyz="0 0 ${lidar_z_offset}" rpy="0 0 0"/>
   </joint>
   <!-- LiDAR Gazebo plugin -->
@@ -136,5 +138,5 @@
     </sensor>
   </gazebo>
-  <!-- ==================== Camera (QR okuma için) ==================== -->
+  <!-- ==================== Camera (QR scanning) ==================== -->
   <link name="camera_link">
     <visual>
@@ -156,5 +158,5 @@
     <parent link="base_link"/>
     <child  link="camera_link"/>
-    <origin xyz="0.13 0 ${base_height/2 + 0.08}" rpy="0 0 0"/>
+    <origin xyz="0.11 0 0.10" rpy="0 0 0"/>
   </joint>
   <link name="camera_optical_link"/>
@@ -190,5 +192,5 @@
     <visual>
       <geometry>
-        <box size="0.22 0.18 0.01"/>
+        <box size="0.18 0.14 0.01"/>
       </geometry>
       <material name="orange">
@@ -198,5 +200,5 @@
     <collision>
       <geometry>
-        <box size="0.22 0.18 0.01"/>
+        <box size="0.18 0.14 0.01"/>
       </geometry>
     </collision>
@@ -217,5 +219,5 @@
     <mu2>0.8</mu2>
   </gazebo>
-  <!-- Differential drive plugin (mecanum yaklaşımı için) -->
+  <!-- Planar simulation plugin; this is kinematic and not a roller-contact model. -->
   <gazebo>
     <plugin name="mecanum_drive_controller" filename="libgazebo_ros_planar_move.so">

Commit message: Align course game, hardware and ROS stack with 2026-27 project rules

File: src/mecanum_description/urdf/mecanum_amr.urdf.xacro (robot description, xacro)
@@ -7,6 +7,6 @@
   <xacro:property name="base_height" value="0.04"/>
   <xacro:property name="base_mass"   value="3.0"/>
-  <!-- 150.8 mm measured circumference gives a 24.0 mm nominal radius. -->
-  <xacro:property name="wheel_radius" value="0.0240006"/>
+  <!-- Teacher materials specify 65 mm wheels; loaded rolling radius needs calibration. -->
+  <xacro:property name="wheel_radius" value="0.0325"/>
   <xacro:property name="wheel_width"  value="0.04"/>
   <xacro:property name="wheel_mass"   value="0.15"/>
@@ -14,5 +14,5 @@
   <xacro:property name="wheel_y_offset" value="0.0675"/>
   <xacro:property name="wheel_z_offset" value="0.0"/>
-  <xacro:property name="lidar_z_offset" value="0.156"/>
+  <xacro:property name="lidar_z_offset" value="0.105"/>
   <!-- ==================== Macros ==================== -->
   <xacro:macro name="box_inertia" params="m w h d">
